File: pcb/p2000t-ram-expansion-board/p2000t-ram-expansion-board.kicad_sch (KiCad schematic)
At the start: 27 parts, among them J1 EXPANSION BOARD, J2 POWER, J3 TERMINAL, U1 74HC04, U2 CY62256-70PC, U3 74HC00, U4 CY62256-70PC, U5 74HC688, U6 74HC32, U7 74HC173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

Commit message: Board revision 3 (#2)
* Adding 74HC245

* Fixing connection

* Revising board and fixing bugs

* Updating README.md

* Updating schematic

* Replacing images
Parts:
- removed D2, D3, D4: LED, LED_SMD:LED_0805_2012Metric_Pad1.15x1.40mm_HandSolder, symbol Device:LED
- removed R1, R2, R3: R, Resistor_SMD:R_0805_2012Metric_Pad1.20x1.40mm_HandSolder, symbol Device:R
- added C9: 0.1uF, Capacitor_THT:C_Disc_D5.0mm_W2.5mm_P5.00mm, symbol Device:C
- added U8: 74HC245, Package_DIP:DIP-20_W7.62mm_Socket, symbol 74xx:74LS245
- renumbered C9 to C10, U8 to U9
Connections:
- net +5V: now also C9.1, U8.1 (A->B), U8.20 (VCC)
- net A13: now also U9.2 (I0a)
- net D0: now also U8.18 (B0)
- net D1: now also U8.17 (B1)
- net D2: now also U8.16 (B2)
- net D3: now also U8.15 (B3)
- net D4: now also U8.14 (B4)
- net D5: now also U8.13 (B5)
- net D6: now also U8.12 (B6)
- net D7: now also U8.11 (B7)
- net GND: now also C9.2, U8.10 (GND), U8.6 (A4), U8.7 (A5), U8.8 (A6), U8.9 (A7); no longer U3.4, U3.5, U9.2 (I0a)
- net S0: now also U8.2 (A0)
- net S1: now also U8.3 (A1)
- net S2: now also U8.4 (A2)
- net ~{CS1}: now also U3.6; no longer U6.11
- net ~{RD}: now also U6.12
- net ~{REN}: now also U1.11; no longer U6.13
- net at U1.10: now also U3.5; no longer U6.12
- net ~{P=Q}: now reaches U5.19 (P=R), U6.4
- net ~{P=Q}: now also U6.13
- net S3: now reaches U7.6 (Q3)
- net S3: now also U8.5 (A3)
- net at U3.3, U6.1: now also U3.4; no longer U1.11
- new net: U6.11, U8.19 (CE)
- no-connect marks 13 -> 11
Other:
- note added: "ADDR >= 0xE000, then both A13 and A14 are high"
- note added: "~(S1 | S2) | ~(A13 & A14)"
- note added: "~{(S1 | S2) & (A13 & A14)}"
- note removed: "Address is at least 0xE000, then both A13 and A14 are high"
- note removed: "Bank LEDS (for debugging purposes)"
- note removed: "Unused gates tied to GND"
- moved on the sheet: U1C, U1D, U1E, U3A, U3B, U3C, U6A, U6C, U6D
