File: pcb/p2000t-ram-expansion-board/p2000t-ram-expansion-board.kicad_sch (KiCad schematic)
At the start: 23 parts, among them J1 EXPANSION BOARD, J2 POWER, J3 TERMINAL, U1 74HC04, U2 CY62256-70PC, U3 74HC00, U4 CY62256-70PC, U5 74HC688, U6 74HC32, U7 74HC173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

Commit message: Fixing connection
Connections:
- net A13: now also U9.2 (I0a)
- net GND: no longer U9.2 (I0a)
Changed lines of the file:
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@@
+    )
+  )
+  (global_label "A13" (shape input) (at 227.33 37.465 180) (fields_autoplaced)
+    (effects (font (size 1 1)) (justify right))
+    (property "Intersheet References" "${INTERSHEET_REFS}" (id 0) (at 222.6681 37.5275 0)
+      (effects (font (size 1 1)) (justify right) hide)
     )
   )
@@
     )
     (property "Datasheet" "" (id 3) (at 165.735 179.705 0)
-      (effects (font (size 1.27 1.27)) hide)
-    )
-    (pin "1")
-  )
-  (symbol (lib_id "power:GND") (at 227.33 37.465 270) (unit 1)
-    (in_bom yes) (on_board yes)
-    (property "Reference" "#PWR047" (id 0) (at 220.98 37.465 0)
-      (effects (font (size 1.27 1.27)) hide)
-    )
-    (property "Value" "GND" (id 1) (at 220.345 37.465 90)
-      (effects (font (size 1.27 1.27)) (justify left))
-    )
-    (property "Footprint" "" (id 2) (at 227.33 37.465 0)
-      (effects (font (size 1.27 1.27)) hide)
-    )
-    (property "Datasheet" "" (id 3) (at 227.33 37.465 0)
       (effects (font (size 1.27 1.27)) hide)
     )
@@
       (reference "#PWR046") (unit 1) (value "GND") (footprint "")
     )
-    (path "/174e448f-68cc-4579-b8da-d300cab8464d"
-      (reference "#PWR047") (unit 1) (value "GND") (footprint "")
-    )
     (path "/61fa287c-bcbb-4d71-8ae2-e91e01adf32a"

Commit message: Revising board and fixing bugs
Connections:
- no-connect marks 12 -> 11
Changed lines of the file:
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@@
   (no_connect (at 46.355 70.485))
   (no_connect (at 33.655 80.645))
-  (no_connect (at 325.755 129.54))
   (no_connect (at 33.655 78.105))
   (no_connect (at 46.355 75.565))
@@
   (symbol (lib_id "74xx:74LS245") (at 201.295 108.585 90) (unit 1)
     (in_bom yes) (on_board yes)
-    (property "Reference" "U8" (id 0) (at 221.615 105.0036 90))
-    (property "Value" "74HC245" (id 1) (at 212.725 99.695 90))
+    (property "Reference" "U8" (id 0) (at 197.7136 88.265 90))
+    (property "Value" "74HC245" (id 1) (at 213.233 99.06 90))
     (property "Footprint" "Package_DIP:DIP-20_W7.62mm_Socket" (id 2) (at 201.295 108.585 0)
       (effects (font (size 1.27 1.27)) hide)

Commit message: Small fixes in schematic
Connections:
- net ~{P=Q}: no longer U5.19 (P=R), U6.4
- new net ~{P=R}: U5.19 (P=R), U6.4
Other:
- note added: "Because of timing contraints, ~{WR} needs to be combined with ~{P=R}"
- note added: "Tie unused gates to GND"
- note removed: "Because of timing contraints, ~{WR} needs to be combined with ~{P=Q}"
Changed lines of the file:
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@@
     (title "P2000T RAM expansion board")
     (date "2023-11-16")
-    (rev "2")
+    (rev "3")
   )
   (junction (at 201.295 125.73) (diameter 0) (color 0 0 0 0)
@@
     (stroke (width 0) (type default) (color 0 0 0 0))
   )
+  (polyline (pts (xy 85.09 179.07) (xy 85.09 196.85))
+    (stroke (width 0) (type default) (color 0 0 0 0))
+  )
   (wire (pts (xy 227.33 61.595) (xy 227.33 62.865))
     (stroke (width 0) (type default) (color 0 0 0 0))
@@
   )
   (wire (pts (xy 166.37 177.165) (xy 164.465 177.165))
+    (stroke (width 0) (type default) (color 0 0 0 0))
+  )
+  (polyline (pts (xy 114.3 179.07) (xy 85.09 179.07))
     (stroke (width 0) (type default) (color 0 0 0 0))
   )
@@
     (effects (font (size 1.27 1.27)) (justify left bottom))
   )
-  (text "Because of timing\ncontraints, ~{WR}\nneeds to be combined\nwith ~{P=Q}"
+  (text "Because of timing\ncontraints, ~{WR}\nneeds to be combined\nwith ~{P=R}"
     (at 175.26 74.676 0)
     (effects (font (size 1.27 1.27)) (justify left bottom))
@@
   )
   (text "32 kb static memory" (at 27.305 124.841 0)
+    (effects (font (size 1.27 1.27)) (justify left bottom))
+  )
+  (text "Tie unused gates to GND" (at 86.36 196.85 0)
     (effects (font (size 1.27 1.27)) (justify left bottom))
   )
@@
     )
   )
-  (global_label "~{P=Q}" (shape input) (at 143.51 62.23 270) (fields_autoplaced)
+  (global_label "~{P=R}" (shape input) (at 143.51 62.23 270) (fields_autoplaced)
     (effects (font (size 1.27 1.27)) (justify right))
-    (property "Intersheet References" "${INTERSHEET_REFS}" (id 0) (at 143.4306 68.816 90)
+    (property "Intersheet References" "${INTERSHEET_REFS}" (id 0) (at 143.4306 68.7555 90)
       (effects (font (size 1.27 1.27)) (justify right) hide)
     )

Commit message: Revising PCBs
Other:
- title: P2000T RAM expansion board -> Philips P2000T 64kb memory expansion board
