File: pcb/p2000t-ram-expansion-board/p2000t-ram-expansion-board.kicad_pcb (KiCad board)
At the start: 2 copper layers, 110 x 68.1 mm, 23 parts, among them J1 EXPANSION BOARD, J2 POWER, J3 TERMINAL, U1 74HC04, U2 CY62256-70PC, U3 74HC00, U4 CY62256-70PC, U5 74HC688, U6 74HC32, U7 74HC173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

Commit message: Fixing connection
Parts:
- moved C10 5.04 mm to (123.8, 24.1), turned to 180 degrees
Connections:
- U9 pad 2: GND -> A13
Routing:
- net GND: track 0.00 -> 703.6 mm
- net +5V: track 0.00 -> 569.0 mm
- net D0: track 0.00 -> 153.1 mm, vias 0 -> 1
- net A5: track 0.00 -> 152.2 mm
- net A13: track 0.00 -> 150.0 mm, vias 0 -> 6
- net D2: track 0.00 -> 140.3 mm
- net D1: track 0.00 -> 136.4 mm
- net D6: track 0.00 -> 131.0 mm
- net A4: track 0.00 -> 123.9 mm
- net D3: track 0.00 -> 119.2 mm
- net A7: track 0.00 -> 109.1 mm
- net ~{RD}: track 0.00 -> 106.0 mm
- net D7: track 0.00 -> 104.9 mm, vias 0 -> 1
- net D4: track 0.00 -> 104.8 mm
- net A3: track 0.00 -> 104.7 mm
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Other:
- board text added: "rev3"
- board text removed: "rev2"

Commit message: Revising board and fixing bugs
Parts:
- added REF**: OSHW-Logo2_9.8x8mm_SilkScreen, Symbol:OSHW-Logo2_9.8x8mm_SilkScreen, F.Cu at (109.2, 79.5)
- added REF**: OSHW-Logo2_9.8x8mm_SilkScreen, Symbol:OSHW-Logo2_9.8x8mm_SilkScreen, B.Cu at (109.2, 79.5)
- moved U2 45.7 mm to (31.8, 70.1)
- moved U4 45.7 mm to (77.5, 69.8)
Routing:
- net A14_1: track 85.8 -> 26.1 mm, vias 1 -> 0
- net A5: track 152.2 -> 107.3 mm, vias 0 -> 1
- net ~{CS1}: track 10.6 -> 54.0 mm, vias 0 -> 1
- net A13_1: track 54.6 -> 18.4 mm, vias 1 -> 0
- net A13_2: track 9.80 -> 43.1 mm, vias 0 -> 1
- net A1: track 85.3 -> 118.1 mm
- net A7: track 109.1 -> 139.8 mm
- net A6: track 101.8 -> 132.1 mm
- net A2: track 99.5 -> 125.3 mm, vias 1 -> 0
- net ~{CS2}: track 62.2 -> 36.7 mm, vias 0 -> 1
- net D6: track 131.0 -> 107.6 mm
- net A14_2: track 34.3 -> 57.5 mm, vias 0 -> 2
- net D5: track 102.7 -> 125.4 mm, vias 0 -> 2
- net GND: track 703.6 -> 726.2 mm
- net A4: track 123.9 -> 101.7 mm, vias 0 -> 1
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Other:
- board text added: "0xA000-0xDFFF + BANKS 0-1"
- board text added: "BANKS 2-5"

Commit message: Revising PCBs
Parts:
- removed REF** (x2): OSHW-Logo2_9.8x8mm_SilkScreen, Symbol:OSHW-Logo2_9.8x8mm_SilkScreen
- added LOGO1: OSHW-Logo2_14.6x12mm_Copper_AND_Mask, components:OSHW-Logo2_14.6x12mm_Copper_AND_Mask, F.Cu at (108.5, 80.0)
Routing:
- net A5: track 107.3 -> 115.6 mm
- net A4: track 101.7 -> 106.6 mm
- net A3: track 126.2 -> 130.8 mm
- net A2: track 125.3 -> 127.1 mm
Other:
- board text added: "rev4"
