File: pcb/p2000t-ram-expansion-board-1056kb/p2000t-ram-expansion-board-1056kb.kicad_sch (KiCad schematic)
At the start: 23 parts, among them J1 EXPANSION BOARD, J2 POWER, J3 TERMINAL, U1 74HC04, U2 AS6C4008-55PCN, U3 74HC00, U4 CY62256-70PC, U5 74HC688, U6 74HC32, U7 74HC273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

Commit message: Storing before routing
Connections:
- net GND: now also U1.1, U1.11
- net S6: now also U3.5; no longer U1.11
- net ~{RES}: now also U7.1 (~{Mr}); no longer U1.1
- net at U1.10: no longer U3.5
- net RES: no longer names the net of U1.2
- net RES: no longer U7.1 (~{Mr})
- no-connect marks 10 -> 12
Other:
- note removed: "Active high reset needed for 74HC173"
- moved on the sheet: C2, U1A, U1E, U4

Commit message: Revising PCBs
Parts:
- J1: value EXPANSION BOARD -> EXPANSION PORT
