File: pcb/p2000t-ram-expansion-board-2080kb/p2000t-ram-expansion-board-2080kb.kicad_sch (KiCad schematic)
At the start: 23 parts, among them J1 EXPANSION PORT, J2 POWER, J3 TERMINAL, U1 74HC04, U2 AS6C4008-55PCN, U3 74HC00, U4 CY62256-70PC, U5 74HC688, U6 74HC32, U7 74HC273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

Commit message: Version 2080kb (#6)
* Initial commit

* Adding gerbers

* Fixing bug in wiring

* Fixing another bug 74HC74

* Changing size

* Revising PCBs
Parts:
- added C11, C12, C13, C14: 0.1uF, Capacitor_THT:C_Disc_D5.0mm_W2.5mm_P5.00mm, symbol Device:C
- added U10, U11: AS6C4008-55PCN, Package_DIP:DIP-32_W15.24mm_Socket, symbol Memory_RAM:AS6C4008-55PCN
- added U12: 74HC138, Package_DIP:DIP-16_W7.62mm_Socket, symbol 74xx:74LS138
- added U13: 74HC74, Package_DIP:DIP-14_W7.62mm_Socket, symbol 74xx:74HC74
- J1: value EXPANSION PORT -> EXPANSION BOARD
Connections:
- net +5V: now also C11.1, C12.1, C13.1, C14.1, U10.32 (VCC), U11.32 (VCC), U12.16 (VCC), U12.6 (E3), U13.10 (~{S}), U13.14 (VCC), U13.4 (~{S})
- net A0: now also U3.4, U6.10, U10.12 (A0), U11.12 (A0); no longer U5.2 (P0)
- net A1: now also U10.11 (A1), U11.11 (A1)
- net A10: now also U10.23 (A10), U11.23 (A10)
- net A11: now also U10.25 (A11), U11.25 (A11)
- net A12: now also U10.4 (A12), U11.4 (A12)
- net A2: now also U10.10 (A2), U11.10 (A2)
- net A3: now also U10.9 (A3), U11.9 (A3)
- net A4: now also U10.8 (A4), U11.8 (A4)
- net A5: now also U10.7 (A5), U11.7 (A5)
- net A6: now also U10.6 (A6), U11.6 (A6)
- net A7: now also U10.5 (A7), U11.5 (A7)
- net A8: now also U10.27 (A8), U11.27 (A8)
- net A9: now also U10.26 (A9), U11.26 (A9)
- net D0: now also U10.13 (DQ0), U11.13 (DQ0), U13.2 (D)
- net D1: now also U10.14 (DQ1), U11.14 (DQ1), U13.12 (D)
- net D2: now also U10.15 (DQ2), U11.15 (DQ2)
- net D3: now also U10.17 (DQ3), U11.17 (DQ3)
- net D4: now also U10.18 (DQ4), U11.18 (DQ4)
- net D5: now also U10.19 (DQ5), U11.19 (DQ5)
- net D6: now also U10.20 (DQ6), U11.20 (DQ6)
- net D7: now also U10.21 (DQ7), U11.21 (DQ7)
- net GND: now also U5.2 (P0), C11.2, C12.2, C13.2, C14.2, U10.16 (VSS), U11.16 (VSS), U12.3 (A2), U12.8 (GND), U13.7 (GND); no longer U1.1
- net S0: now also U10.28 (A13), U11.28 (A13)
- net S1: now also U10.3 (A14), U11.3 (A14)
- net S2: now also U10.31 (A15), U11.31 (A15)
- net S3: now also U10.2 (A16), U11.2 (A16)
- net S4: now also U10.30 (A17), U11.30 (A17)
- net S5: now also U10.1 (A18), U11.1 (A18)
- net S6: now also U12.1 (A0); no longer U3.5, U6.10
- net S7: now also U12.2 (A1); no longer U4.1 (A14)
- net ~{CS1}: now also U12.15 (O0); no longer U6.8
- net ~{CS2}: now also U12.14 (O1); no longer U3.6
- net ~{CS3}: now also U10.22 (CE#), U12.13 (O2); no longer U3.3, U4.20 (~{CS})
- net ~{P=R}: now also U1.9, U6.9; no longer U6.4
- net ~{RD}: now also U10.24 (OE#), U11.24 (OE#)
- net ~{REN}: now also U12.4 (E1); no longer U6.2
- net ~{RES}: now also U13.1 (~{R}), U13.13 (~{R})
- net ~{WR}: now also U6.2, U10.29 (WE#), U11.29 (WE#)
- net at U1.8: now also U3.5; no longer U3.4
- net at U1.2: now also U13.11 (C), U13.3 (C)
- net at U3.1, U3.8: now also U12.5 (E2); no longer U6.1
- new net: U3.6, U6.1
- new net: U6.4, U6.8
- new net: U1.1, U6.3
- new net RAMS0: U13.5 (Q), U4.1 (A14)
- new net ~{CS4}: U11.22 (CE#), U12.12 (O3)
- new net ~{CS5}: U3.3, U4.20 (~{CS})
- no-connect marks 12 -> 18
Other:
- note added: "0x94 | 0x95"
- note added: "Currently not used"
- note added: "Port number 0x94 or 0x95 select D-type flip-flop 0x94 = 1001 0100 0x95 = 1001 0101"
- note added: "Whether one of the expansion RAM slots need to be accessed."
- note added: "Writeable on port 0x94"
- note added: "Writeable on port 0x95"
- note removed: "0x94"
- note removed: "Port number 0x94 selects D-type flip-flop 0x94 = 1001 0100"
- note removed: "Whether one of the two RAM chips should be set active"
- title: P2000T RAM expansion board -> Philips P2000T Memory Expansion 2Mb+
- moved on the sheet: C2, C4, U1A, U1C, U1D, U1E, U3A, U3B, U3C, U4, U6A, U6C
